Commit message: dev container + square chassis

File: src/edna_description/urdf/parts/square_chassis.xacro (robot description, xacro)
@@ -19,5 +19,5 @@
         <origin xyz="0.061605 0.53866 -0.34976" rpy="${pi / 2} 0 0" />
         <geometry>
-          <mesh filename="package://edna_description/meshes/SwerveChassis.stl" scale="0.001 0.001 0.001" />
+          <mesh filename="package://edna_description/meshes/RiftChassis.stl" scale="0.001 0.001 0.001" />
         </geometry>
         <material name="red"/>

Commit message: chassis

File: src/edna_description/urdf/parts/square_chassis.xacro (robot description, xacro)
@@ -2,10 +2,10 @@
 <robot xmlns:xacro="http://www.ros.org/wiki/xacro">
   <!-- Chassis Properties -->
-  <xacro:property name="chassis_length" value=".7366" />
-  <xacro:property name="chassis_width" value=".7366" />
-  <xacro:property name="chassis_height" value="0.05588" />
-  <xacro:property name="chassis_weight" value="85" />
-  <xacro:property name="bumper_length" value="0.8128" />
-  <xacro:property name="bumper_width" value="0.8128" />
+  <xacro:property name="chassis_length" value="0.6604" />
+  <xacro:property name="chassis_width" value="0.6604" />
+  <xacro:property name="chassis_height" value="0.0508" />
+  <xacro:property name="chassis_weight" value="11.7934" />
+  <xacro:property name="bumper_length" value="0.762" />
+  <xacro:property name="bumper_width" value="0.762" />
   <xacro:property name="bumper_height" value="0.127" />
   <xacro:property name="bumper_weight" value="6.80388555" />
@@ -14,8 +14,8 @@
     <link name="${prefix}_chassis_link">
       <xacro:inertial_box mass="${chassis_weight}" x="${chassis_length}" y="${chassis_width}" z="${chassis_height}">
-        <origin xyz="0 0 ${chassis_height/2}" rpy="0 0 0" />
+        <origin xyz="0 0 0" rpy="0 0 0" />
       </xacro:inertial_box>
       <visual>
-        <origin xyz="0.061605 0.53866 -0.34976" rpy="${pi / 2} 0 0" />
+        <origin xyz="0 0 ${chassis_height/2}" rpy="0 0 ${pi/2}" />
         <geometry>
           <mesh filename="package://edna_description/meshes/RiftChassis.stl" scale="0.001 0.001 0.001" />
@@ -24,5 +24,5 @@
       </visual>
       <collision>
-        <origin xyz="0 0 ${chassis_height/2}" rpy="0 0 0" />
+        <origin xyz="0 0 0" rpy="0 0 0" />
         <geometry>
           <box size="${chassis_length} ${chassis_width} ${chassis_height} " />

File: src/edna_description/urdf/parts/swerve_axle.xacro (robot description, xacro)
@@ -35,5 +35,5 @@
         <link name="${prefix}_wheel_link">
             <visual>
-                <origin xyz="0 -${wheel_pos_y} 0" rpy="0 ${pi/4} ${pi/2}" />
+                <origin xyz="0 ${wheel_pos_y} 0" rpy="${pi} ${pi/4} ${pi/2}" />
                 <geometry>
                     <mesh filename="package://edna_description/meshes/SwerveWheel.stl" scale="0.001 0.001 0.001" />

File: src/edna_description/urdf/robots/edna.urdf.xacro (robot description, xacro)
@@ -18,5 +18,5 @@
   <xacro:include filename="$(find edna_description)/urdf/parts/intake.xacro" />
   <!-- Axle Position Variables -->
-  <xacro:property name="axle_pos" value="${301.625 / 1000}" />
+  <xacro:property name="axle_pos" value="0.261523" />
   <xacro:property name="axle_pos_z" value="${69.056 / 1000}" />
   <xacro:property name="elevator_middle_distance" value = ".457" />
@@ -53,12 +53,12 @@
   </xacro:swerve_axle>
   <!-- Sensors -->
-  <xacro:zed_camera prefix="zed2i" model="zed2i" parent="swerve_chassis_link">
+  <!-- <xacro:zed_camera prefix="zed2i" model="zed2i" parent="swerve_chassis_link">
     <origin xyz="${cam_pos}" rpy="0 0 0" />
-  </xacro:zed_camera>
+  </xacro:zed_camera> -->
   <!-- <xacro:lidar prefix="lidar" parent="swerve_chassis_link" radius="0.035" length="0.025">
     <origin xyz="${lidar_pos}" rpy="0 0 0" />
   </xacro:lidar> -->
   <!-- Arm -->
-  <xacro:property name="elevator_leg_z" value="0.527"/>
+  <!-- <xacro:property name="elevator_leg_z" value="0.527"/>
   <xacro:elevator_leg prefix="arm" parent="swerve_chassis_link">
     <origin xyz = "0.1905 0 ${elevator_leg_z/2 + 0.03}" rpy = "0 0 0"/>
@@ -66,14 +66,14 @@
   <xacro:back_leg prefix="arm" parent="swerve_chassis_link">
     <origin xyz = "-${chassis_length/2 - each_leg_width * 2} 0 ${chassis_height}" rpy = "0 0 0" />
-  </xacro:back_leg>
+  </xacro:back_leg> -->
   <!--Elevator-->
-  <xacro:elevator prefix="elevator" parent="arm_back_leg_link">
+  <!-- <xacro:elevator prefix="elevator" parent="arm_back_leg_link">
     <origin xyz = "-.03 -${elevator_middle_distance / 2} ${back_leg_height - .0215}" rpy = "0 0 0" />
-  </xacro:elevator>
+  </xacro:elevator> -->
   <!-- Top Slider + Gripper -->
-  <xacro:property name= "slider_pos" value = "0.330 ${elevator_middle_distance / 2} ${slider_block_height/2}" />
+  <!-- <xacro:property name= "slider_pos" value = "0.330 ${elevator_middle_distance / 2} ${slider_block_height/2}" />
   <xacro:slider prefix="top" parent="elevator_outer_2_link">
     <origin xyz = "${slider_pos}" rpy = "0 0 0" />
-  </xacro:slider>
+  </xacro:slider> -->
   <!-- Control -->
   <xacro:swerve_drive_control plugin="$(arg hw_interface_plugin)"/>

Commit message: Rotated wheels to correct rotation and moved collision for chassis up

File: src/edna_description/urdf/parts/square_chassis.xacro (robot description, xacro)
@@ -24,5 +24,5 @@
       </visual>
       <collision>
-        <origin xyz="0 0 0" rpy="0 0 0" />
+        <origin xyz="0 0 ${chassis_height/2}" rpy="0 0 0" />
         <geometry>
           <box size="${chassis_length} ${chassis_width} ${chassis_height} " />

File: src/edna_description/urdf/parts/swerve_axle.xacro (robot description, xacro)
@@ -35,5 +35,5 @@
         <link name="${prefix}_wheel_link">
             <visual>
-                <origin xyz="0 ${wheel_pos_y} 0" rpy="${pi / 2} 0 -${pi / 4}" />
+                <origin xyz="0 ${wheel_pos_y} 0" rpy="${pi / 2} 0 ${pi / 4}" />
                 <geometry>
                     <mesh filename="package://edna_description/meshes/SwerveWheel.stl" scale="0.001 0.001 0.001" />
