Commit message: Changed robot color, added intake and versa rollerbars

File: src/edna_description/urdf/parts/intake.xacro (robot description, xacro)
@@ -1,36 +1,34 @@
 <?xml version="1.0" ?>
 <robot xmlns:xacro="http://www.ros.org/wiki/xacro">
-    <xacro:property name="intake_block_height" value="0.0508" />
-    <xacro:property name="intake_block_length" value="0.449834" />
-    <xacro:property name="intake_block_width" value="0.4064" />
-  <xacro:macro name="intake" params="prefix parent *origin">
-    <link name = "${prefix}_intake_link">
-        <xacro:inertial_box mass = "1" x = "${intake_block_length}" y = "${intake_block_length}" z = "${intake_block_height}">
-            <origin xyz = "0 0 0" rpy = "0 0 0"/>
-        </xacro:inertial_box>
+    <xacro:macro name="intake" params="parent *origin">
+    <link name="intake_link">
         <visual>
-            <origin xyz = "${intake_block_length-0.04} ${intake_block_width/2} -0.0508" rpy = "${pi/2} 0 0"/>
-            <geometry>
-                <mesh filename = "package://edna_description/meshes/Front_Intake_V2.stl" scale="0.001 0.001 0.001"/>
-            </geometry>
-            <material name = "blue"/>
+        <origin xyz="0 0 0" rpy="0 0 0" />
+        <geometry>
+            <mesh filename="package://edna_description/meshes/RiftIntake.stl" scale="1 1 1" />
+        </geometry>
+        <material name="blue"/>
         </visual>
         <collision>
-            <origin xyz = "${intake_block_length/2 - 0.03} 0 0" rpy = "0 0 0"/>
-            <geometry>
-                <box size="${intake_block_length} ${intake_block_width} ${intake_block_height}"/>
-            </geometry>
+            <!-- TODO: Add collision to sides with rectangles -->
         </collision>
     </link>
-    <joint name="${prefix}_intake_joint" type="revolute">
+    <xacro:versaroller prefix="0" parent="intake_link">
+        <origin xyz="0 .10836 -0.008356" rpy="0 ${pi/2} 0" />
+    </xacro:versaroller>
+    <xacro:versaroller prefix="1" parent="intake_link">
+        <origin xyz="0.000201 0.045509 0.028214" rpy="0 ${pi/2} 0" />
+    </xacro:versaroller>
+    <xacro:versaroller prefix="2" parent="intake_link">
+        <origin xyz="-0.000036 0.088642 -0.08196" rpy="0 ${pi/2} 0" />
+    </xacro:versaroller>
+    <xacro:versaroller prefix="3" parent="intake_link">
+        <origin xyz="-0.000053 0.0254 -0.045558" rpy="0 ${pi/2} 0" />
+    </xacro:versaroller>
+    <joint name="intake_joint" type="fixed">
+        <parent link="${parent}"/>
+        <child link="intake_link"/>
         <xacro:insert_block name="origin" />
-        <parent link="${parent}"/>
-        <child link="${prefix}_intake_link"/>
-        <axis xyz = "0 1 0"/>
-        <limit effort = "100.0" lower = "0" upper = "${pi/2 - 0.05}" velocity = "1"/>
     </joint>
-    <!-- <xacro:gripper prefix="${prefix}" parent="${prefix}_intake_link">
-        <origin xyz = "${intake_block_length - 0.05} 0 -0.035" rpy = "0 0 0" />
-    </xacro:gripper> -->
-  </xacro:macro>
+    </xacro:macro>
 </robot>

File: src/edna_description/urdf/parts/square_chassis.xacro (robot description, xacro)
@@ -21,5 +21,5 @@
           <mesh filename="package://edna_description/meshes/RiftChassis.stl" scale="0.001 0.001 0.001" />
         </geometry>
-        <material name="red"/>
+        <material name="purple"/>
       </visual>
       <collision>
@@ -30,5 +30,5 @@
       </collision>
     </link>
-    <link name="${prefix}_bumper_link">
+    <!-- <link name="${prefix}_bumper_link">
       <xacro:inertial_box mass="${bumper_weight}" x="${bumper_length}" y="${bumper_width}" z="${bumper_height}">
         <origin xyz="0 0 ${bumper_height/2 + 0.0127}" rpy="0 0 0" />
@@ -47,5 +47,5 @@
         </geometry>
       </collision>
-    </link>
+    </link> -->
     <joint name="${prefix}_chassis_joint" type="fixed">
       <parent link="${parent}" />
@@ -53,9 +53,9 @@
       <xacro:insert_block name="origin" />
     </joint>
-    <joint name="${prefix}_bumper_joint" type="fixed">
+    <!-- <joint name="${prefix}_bumper_joint" type="fixed">
       <parent link="${parent}" />
       <child link="${prefix}_bumper_link" />
       <xacro:insert_block name="origin" />
-    </joint>
+    </joint> -->
   </xacro:macro>
 </robot>

File: src/edna_description/urdf/robots/edna.urdf.xacro (robot description, xacro)
@@ -17,4 +17,5 @@
   <xacro:include filename="$(find edna_description)/urdf/parts/slider.xacro" />
   <xacro:include filename="$(find edna_description)/urdf/parts/intake.xacro" />
+  <xacro:include filename="$(find edna_description)/urdf/parts/versaroller.xacro" />
   <!-- Axle Position Variables -->
   <xacro:property name="axle_pos" value="0.261523" />
@@ -39,4 +40,7 @@
     <origin xyz="0 0 0" rpy="0 0 0" />
   </xacro:square_chassis>
+  <xacro:intake parent="swerve_chassis_link">
+    <origin xyz="0 -0.46 0.09" rpy="0 0 0" />
+  </xacro:intake>
   <!-- Drive Train -->
   <xacro:swerve_axle prefix="front_left" parent="swerve_chassis_link">

File: src/edna_description/urdf/util/materials.xacro (robot description, xacro)
@@ -22,4 +22,7 @@
     <color rgba="${255/255} ${215/255} ${0/255} 1" />
   </material>
+  <material name="purple">
+    <color rgba="${127/255} 0 ${127/255} 1" />
+  </material>
   <material name="orange">
     <color rgba="${243/255} ${135/255} ${47/255} 1" />

Commit message: Intake collision and side axis fixed

File: src/edna_description/urdf/parts/intake.xacro (robot description, xacro)
@@ -4,12 +4,30 @@
     <link name="intake_link">
         <visual>
-        <origin xyz="0 0 0" rpy="0 0 0" />
-        <geometry>
-            <mesh filename="package://edna_description/meshes/RiftIntake.stl" scale="1 1 1" />
-        </geometry>
-        <material name="blue"/>
+            <origin xyz="0 0 0" rpy="0 0 0" />
+            <geometry>
+                <mesh filename="package://edna_description/meshes/RiftIntake.stl" scale="1 1 1" />
+            </geometry>
+            <material name="blue"/>
         </visual>
+        <!-- Front plate collision -->
         <collision>
-            <!-- TODO: Add collision to sides with rectangles -->
+            <origin xyz="0 ${0.0254/2} 0" rpy="0 0 0" />
+            <geometry>
+                <box size="0.575 0.0254 0.102" />
+            </geometry>
+        </collision>
+        <!-- +Y side collision -->
+        <collision>
+            <origin xyz="${0.575/2+0.038/2} 0.065 0.007" rpy="0 0 0" />
+            <geometry>
+                <box size="0.038 0.127 0.22" />
+            </geometry>
+        </collision>
+        <!-- -Y side collision -->
+        <collision>
+            <origin xyz="${-0.575/2-0.038/2} 0.065 0.007" rpy="0 0 0" />
+            <geometry>
+                <box size="0.038 0.127 0.22" />
+            </geometry>
         </collision>
     </link>

File: src/edna_description/urdf/robots/edna.urdf.xacro (robot description, xacro)
@@ -40,6 +40,7 @@
     <origin xyz="0 0 0" rpy="0 0 0" />
   </xacro:square_chassis>
+  <!-- Intake -->
   <xacro:intake parent="swerve_chassis_link">
-    <origin xyz="0 -0.46 0.09" rpy="0 0 0" />
+    <origin xyz="0.46 0 0.09" rpy="0 0 ${pi/2}" />
   </xacro:intake>
   <!-- Drive Train -->
