Commit message: not finsh

File: src/edna_description/urdf/parts/shooter.xacro (robot description, xacro)
@@ -1,10 +1,18 @@
 <?xml version="1.0" ?>
+<!--add 2 cylinders, with collisions wheel radius, and 4 revolute joints with panel-->
 <robot xmlns:xacro="http://www.ros.org/wiki/xacro">
-    <xacro:property name="slider_block_height" value="0.079" />
-    <xacro:property name="slider_block_length" value="${gripper_bar_length}" />
-    <xacro:property name="slider_block_width" value="${elevator_middle_distance}" />
-  <xacro:macro name="slider" params="prefix parent *origin">
-    <link name = "${prefix}_slider_link">
-        <xacro:inertial_box mass = "0.90718474" x = "${slider_block_length}" y = "${slider_block_width}" z = "${slider_block_height}">
+    <xacro:property name="panel_height" value="0.4266184" /> <!--also serves as back panel height-->
+    <xacro:property name="panel_width" value="0.254" />
+    <xacro:property name="panel_thick" value="0.00635" />
+    <xacro:property name="panel_weight" value="0.5715264" />
+    <xacro:property name="back_panel_length" value="0.364" />
+    <xacro:property name="back_panel_thick" value="0.021" />
+    <xacro:property name="wheel_radius" value="0.0505" />
+    <xacro:property name="wheel_length" value="0.025" /> <!--but really thickness-->
+    <xacro:property name="wheel_mass" value="0.11566605" /> <!--not the most accurate, but issok-->
+    <!--<xacro:property name="back_panel_weight" value=""/>-->
+  <xacro:macro name="shooter" params="prefix parent *origin">
+    <link name = "shooter_leftPanel_link">
+        <xacro:inertial_box mass = "${panel_weight}" x = "${panel_width}" y = "${panel_height}" z = "${panel_thick}">
             <origin xyz = "0 0 0" rpy = "0 0 0"/>
         </xacro:inertial_box>
@@ -12,5 +20,5 @@
             <origin xyz = "0 0 0" rpy = "0 0 0"/>
             <geometry>
-                <box size="${slider_block_length} ${slider_block_width} ${slider_block_height}"/>
+                <box size="${panel_width} ${panel_height} ${panel_thick}"/>
             </geometry>
             <material name = "blue"/>
@@ -19,18 +27,158 @@
             <origin xyz = "0 0 0" rpy = "0 0 0"/>
             <geometry>
-                <box size="${slider_block_length} ${slider_block_width} ${slider_block_height}"/>
+                <box size="${panel_width} ${panel_height} ${panel_thick}"/>
             </geometry>
         </collision>
     </link>
-    <joint name="${prefix}_slider_joint" type="prismatic">
-        <xacro:insert_block name="origin" />
-        <parent link="${parent}"/>
-        <child link="${prefix}_slider_link"/>
-        <axis xyz = "1 0 0"/>
-        <limit effort = "100.0" lower = "0" upper = "0.3" velocity = "1"/>
+    <link name = "shooter_rightPanel_link">
+         <xacro:inertial_box mass = "${panel_weight}" x = "${panel_width}" y = "${panel_height}" z = "${panel_thick}">
+            <origin xyz = "0 0 0" rpy = "0 0 0"/>
+        </xacro:inertial_box>
+        <visual>
+            <origin xyz = "0 0 0" rpy = "0 0 0"/>
+            <geometry>
+                <box size="${panel_width} ${panel_height} ${panel_thick}"/>
+            </geometry>
+            <material name = "blue"/>
+        </visual>
+        <collision>
+            <origin xyz = "0 0 0" rpy = "0 0 0"/>
+            <geometry>
+                <box size="${panel_width} ${panel_height} ${panel_thick}"/>
+            </geometry>
+        </collision>
+    </link>
+    <link name = "shooter_backPanel_link">
+        <xacro:inertial_box mass = "0.02" x = "${back_panel_length}" y = "${panel_height}" z = "${back_panel_thick}">
+            <origin xyz = "0 0 0" rpy = "0 0 0"/>
+        </xacro:inertial_box>
+        <visual>
+            <origin xyz = "0 0 0" rpy = "0 0 0"/>
+            <geometry>
+                <box size="${back_panel_width} ${panel_height} ${back_panel_thick}"/>
+            </geometry>
+            <material name = "blue"/>
+        </visual>
+        <collision>
+            <origin xyz = "0 0 0" rpy = "0 0 0"/>
+            <geometry>
+                <box size="${back_panel_width} ${panel_height} ${back_panel_thick}"/>
+            </geometry>
+        </collision>
+    </link>
+    <link name = "shooter_frontPanel_link">
+        <xacro:inertial_box mass = "0.02" x = "${back_panel_length}" y = "${panel_height}" z = "${back_panel_thick}">
+            <origin xyz = "0 0 0" rpy = "0 0 0"/>
+        </xacro:inertial_box>
+        <visual>
+            <origin xyz = "0 0 0" rpy = "0 0 0"/>
+            <geometry>
+                <box size="${back_panel_width} ${panel_height} ${back_panel_thick}"/>
+            </geometry>
+            <material name = "blue"/>
+        </visual>
+        <collision>
+            <origin xyz = "0 0 0" rpy = "0 0 0"/>
+            <geometry>
+                <box size="${back_panel_width} ${panel_height} ${back_panel_thick}"/>
+            </geometry>
+        </collision>
+    </link>
+    <link name="${prefix}_wheel_L1_link">
+            <visual>
+                <origin xyz="0 0 0" rpy="${pi / 2} 0 0" />
+                <geometry>
+                    <mesh filename="" scale="0.001 0.001 0.001" />
+                </geometry>
+                <material name="yellow" />
+            </visual>
+            <collision>
+                <origin xyz="0 0 0" rpy="${pi / 2} 0 0"/>
+                <geometry>
+                    <cylinder length="${wheel_length}" radius="${wheel_radius}"/>
+                    <!-- <mesh filename="package://edna_description/meshes/SwerveWheel.stl" scale="0.001 0.001 0.001" /> -->
+                </geometry>
+            </collision>
+            <xacro:inertial_cylinder mass="${wheel_mass}" radius="${wheel_radius}" length="${wheel_length}" >
+                <origin xyz="0 0 0" rpy="${pi / 2} 0 0" />
+            </xacro:inertial_cylinder>
+        </link>
+        <link name="${prefix}_wheel_CL1_link">
+            <visual>
+                <origin xyz="0 0 0" rpy="${pi / 2} 0 0" />
+                <geometry>
+                    <mesh filename="" scale="0.001 0.001 0.001" />
+                </geometry>
+                <material name="yellow" />
+            </visual>
+            <collision>
+                <origin xyz="0 0 0" rpy="${pi / 2} 0 0"/>
+                <geometry>
+                    <cylinder length="${wheel_length}" radius="${wheel_radius}"/>
+                    <!-- <mesh filename="package://edna_description/meshes/SwerveWheel.stl" scale="0.001 0.001 0.001" /> -->
+                </geometry>
+            </collision>
+            <xacro:inertial_cylinder mass="${wheel_mass}" radius="${wheel_radius}" length="${wheel_length}" >
+                <origin xyz="0 0 0" rpy="${pi / 2} 0 0" />
+            </xacro:inertial_cylinder>
+        </link>
+        <link name="${prefix}_wheel_CR1_link">
+            <visual>
+                <origin xyz="0 0 0" rpy="${pi / 2} 0 0" />
+                <geometry>
+                    <mesh filename="" scale="0.001 0.001 0.001" />
+                </geometry>
+                <material name="yellow" />
+            </visual>
+            <collision>
+                <origin xyz="0 0 0" rpy="${pi / 2} 0 0"/>
+                <geometry>
+                    <cylinder length="${wheel_length}" radius="${wheel_radius}"/>
+                    <!-- <mesh filename="package://edna_description/meshes/SwerveWheel.stl" scale="0.001 0.001 0.001" /> -->
+                </geometry>
+            </collision>
+            <xacro:inertial_cylinder mass="${wheel_mass}" radius="${wheel_radius}" length="${wheel_length}" >
+                <origin xyz="0 0 0" rpy="${pi / 2} 0 0" />
+            </xacro:inertial_cylinder>
+        </link>
+        <link name="${prefix}_wheel_R1_link">
+            <visual>
+                <origin xyz="0 0 0" rpy="${pi / 2} 0 0" />
+                <geometry>
+                    <mesh filename="" scale="0.001 0.001 0.001" />
+                </geometry>
+                <material name="yellow" />
+            </visual>
+            <collision>
+                <origin xyz="0 0 0" rpy="${pi / 2} 0 0"/>
+                <geometry>
+                    <cylinder length="${wheel_length}" radius="${wheel_radius}"/>
+                    <!-- <mesh filename="package://edna_description/meshes/SwerveWheel.stl" scale="0.001 0.001 0.001" /> -->
+                </geometry>
+            </collision>
+            <xacro:inertial_cylinder mass="${wheel_mass}" radius="${wheel_radius}" length="${wheel_length}" >
+                <origin xyz="0 0 0" rpy="${pi / 2} 0 0" />
+            </xacro:inertial_cylinder>
+        </link>
+     <joint name="${prefix}_left_joint_back" type="fixed">
+      <parent link="${prefix}shooter_leftPanel_link" />
+      <child link="${prefix}_shooter_backPanel_link" />
+      <xacro:insert_block name="origin" />
     </joint>
-    <xacro:gripper prefix="${prefix}" parent="${prefix}_slider_link">
-        <origin xyz = "0 0 ${slider_block_height/2}" rpy = "0 0 0" />
-    </xacro:gripper>
+    <joint name="${prefix}_right_joint_back" type="fixed">
+      <parent link="${prefix}shooter_rightPanel_link" />
+      <child link="${prefix}_shooter_backPanel_link" />
+      <xacro:insert_block name="origin" />
+    </joint>
+    <joint name="${prefix}_left_joint_front" type="fixed">
+      <parent link="${prefix}shooter_leftPanel_link" />
+      <child link="${prefix}_shooter_frontPanel_link" />
+      <xacro:insert_block name="origin" />
+    </joint>
+    <joint name="${prefix}_right_joint_front" type="fixed">
+      <parent link="${prefix}shooter_rightPanel_link" />
+      <child link="${prefix}_shooter_frontPanel_link" />
+      <xacro:insert_block name="origin" />
+    </joint>
   </xacro:macro>
 </robot>

Commit message: still not finsh deleted meshes and added shoter

File: src/edna_description/urdf/parts/shooter.xacro (robot description, xacro)
@@ -8,10 +8,21 @@
     <xacro:property name="back_panel_length" value="0.364" />
     <xacro:property name="back_panel_thick" value="0.021" />
+    <xacro:property name="back_panel_width" value="0.021" />
     <xacro:property name="wheel_radius" value="0.0505" />
-    <xacro:property name="wheel_length" value="0.025" /> <!--but really thickness-->
-    <xacro:property name="wheel_mass" value="0.11566605" /> <!--not the most accurate, but issok-->
+    <!--<xacro:property name="wheel_length" value="0.025" /> --> <!--but really thickness-->
+    <xacro:property name="wheel_mass" value="${0.11566605*4}" /> <!--not the most accurate, but issok-->
+    <xacro:property name="wheel_length" value="0.363538"/>
     <!--<xacro:property name="back_panel_weight" value=""/>-->
   <xacro:macro name="shooter" params="prefix parent *origin">
-    <link name = "shooter_leftPanel_link">
+    <link name="${prefix}_shooter_link">
+        <visual>
+            <origin xyz="0 0 0" rpy="${pi / 2} 0 0" />
+            <geometry>
+                <mesh filename="package://edna_description/meshes/RIFT_shooter.stl" scale="1 1 1" />
+            </geometry>
+            <material name="red" />
+        </visual>
+    </link>
+    <link name = "${prefix}_shooter_leftPanel_link">
         <xacro:inertial_box mass = "${panel_weight}" x = "${panel_width}" y = "${panel_height}" z = "${panel_thick}">
             <origin xyz = "0 0 0" rpy = "0 0 0"/>
@@ -22,5 +33,5 @@
                 <box size="${panel_width} ${panel_height} ${panel_thick}"/>
             </geometry>
-            <material name = "blue"/>
+            <material name = "red"/>
         </visual>
         <collision>
@@ -31,5 +42,5 @@
         </collision>
     </link>
-    <link name = "shooter_rightPanel_link">
+    <link name = "${prefix}_shooter_rightPanel_link">
          <xacro:inertial_box mass = "${panel_weight}" x = "${panel_width}" y = "${panel_height}" z = "${panel_thick}">
             <origin xyz = "0 0 0" rpy = "0 0 0"/>
@@ -40,5 +51,5 @@
                 <box size="${panel_width} ${panel_height} ${panel_thick}"/>
             </geometry>
-            <material name = "blue"/>
+            <material name = "red"/>
         </visual>
         <collision>
@@ -49,5 +60,5 @@
         </collision>
     </link>
-    <link name = "shooter_backPanel_link">
+    <link name = "${prefix}_shooter_backPanel_link">
         <xacro:inertial_box mass = "0.02" x = "${back_panel_length}" y = "${panel_height}" z = "${back_panel_thick}">
             <origin xyz = "0 0 0" rpy = "0 0 0"/>
@@ -58,5 +69,5 @@
                 <box size="${back_panel_width} ${panel_height} ${back_panel_thick}"/>
             </geometry>
-            <material name = "blue"/>
+            <material name = "red"/>
         </visual>
         <collision>
@@ -67,5 +78,5 @@
         </collision>
     </link>
-    <link name = "shooter_frontPanel_link">
+    <link name = "${prefix}_shooter_frontPanel_link">
         <xacro:inertial_box mass = "0.02" x = "${back_panel_length}" y = "${panel_height}" z = "${back_panel_thick}">
             <origin xyz = "0 0 0" rpy = "0 0 0"/>
@@ -76,5 +87,5 @@
                 <box size="${back_panel_width} ${panel_height} ${back_panel_thick}"/>
             </geometry>
-            <material name = "blue"/>
+            <material name = "red"/>
         </visual>
         <collision>
@@ -85,5 +96,5 @@
         </collision>
     </link>
-    <link name="${prefix}_wheel_L1_link">
+    <link name="${prefix}_wheel_set1_link">
             <visual>
                 <origin xyz="0 0 0" rpy="${pi / 2} 0 0" />
@@ -91,5 +102,5 @@
                     <mesh filename="" scale="0.001 0.001 0.001" />
                 </geometry>
-                <material name="yellow" />
+                <material name="red" />
             </visual>
             <collision>
@@ -104,5 +115,5 @@
             </xacro:inertial_cylinder>
         </link>
-        <link name="${prefix}_wheel_CL1_link">
+        <link name="${prefix}_wheel_set2_link">
             <visual>
                 <origin xyz="0 0 0" rpy="${pi / 2} 0 0" />
@@ -110,5 +121,5 @@
                     <mesh filename="" scale="0.001 0.001 0.001" />
                 </geometry>
-                <material name="yellow" />
+                <material name="red" />
             </visual>
             <collision>
@@ -123,62 +134,53 @@
             </xacro:inertial_cylinder>
         </link>
-        <link name="${prefix}_wheel_CR1_link">
-            <visual>
-                <origin xyz="0 0 0" rpy="${pi / 2} 0 0" />
-                <geometry>
-                    <mesh filename="" scale="0.001 0.001 0.001" />
-                </geometry>
-                <material name="yellow" />
-            </visual>
-            <collision>
-                <origin xyz="0 0 0" rpy="${pi / 2} 0 0"/>
-                <geometry>
-                    <cylinder length="${wheel_length}" radius="${wheel_radius}"/>
-                    <!-- <mesh filename="package://edna_description/meshes/SwerveWheel.stl" scale="0.001 0.001 0.001" /> -->
-                </geometry>
-            </collision>
-            <xacro:inertial_cylinder mass="${wheel_mass}" radius="${wheel_radius}" length="${wheel_length}" >
-                <origin xyz="0 0 0" rpy="${pi / 2} 0 0" />
-            </xacro:inertial_cylinder>
-        </link>
-        <link name="${prefix}_wheel_R1_link">
-            <visual>
-                <origin xyz="0 0 0" rpy="${pi / 2} 0 0" />
-                <geometry>
-                    <mesh filename="" scale="0.001 0.001 0.001" />
-                </geometry>
-                <material name="yellow" />
-            </visual>
-            <collision>
-                <origin xyz="0 0 0" rpy="${pi / 2} 0 0"/>
-                <geometry>
-                    <cylinder length="${wheel_length}" radius="${wheel_radius}"/>
-                    <!-- <mesh filename="package://edna_description/meshes/SwerveWheel.stl" scale="0.001 0.001 0.001" /> -->
-                </geometry>
-            </collision>
-            <xacro:inertial_cylinder mass="${wheel_mass}" radius="${wheel_radius}" length="${wheel_length}" >
-                <origin xyz="0 0 0" rpy="${pi / 2} 0 0" />
-            </xacro:inertial_cylinder>
-        </link>
+    <joint name="${prefix}_wheelset1_joint" type="revolute">
+      <origin xyz = "0 0 0" rpy = "0 0 0" />
+      <parent link="${prefix}_shooter_leftPanel_link"/>
+      <child link="${prefix}_wheel_set1_link"/>
+      <axis xyz = "0 1 0"/>
+      <limit effort="100" lower="-1" upper="1" velocity="2"/>
+    </joint>
+    <joint name="${prefix}_wheelset2_joint" type="revolute">
+      <origin xyz = "0 0 0" rpy = "0 0 0" />
+      <parent link="${prefix}_shooter_leftPanel_link"/>
+      <child link="${prefix}_wheel_set2_link"/>
+      <axis xyz = "0 1 0"/>
+      <limit effort="100" lower="-1" upper="1" velocity="2"/>
+    </joint>
      <joint name="${prefix}_left_joint_back" type="fixed">
-      <parent link="${prefix}shooter_leftPanel_link" />
+      <parent link="${prefix}_shooter_leftPanel_link" />
       <child link="${prefix}_shooter_backPanel_link" />
       <xacro:insert_block name="origin" />
     </joint>
     <joint name="${prefix}_right_joint_back" type="fixed">
-      <parent link="${prefix}shooter_rightPanel_link" />
+      <parent link="${prefix}_shooter_rightPanel_link" />
       <child link="${prefix}_shooter_backPanel_link" />
       <xacro:insert_block name="origin" />
     </joint>
     <joint name="${prefix}_left_joint_front" type="fixed">
-      <parent link="${prefix}shooter_leftPanel_link" />
+      <parent link="${prefix}_shooter_leftPanel_link" />
       <child link="${prefix}_shooter_frontPanel_link" />
       <xacro:insert_block name="origin" />
     </joint>
     <joint name="${prefix}_right_joint_front" type="fixed">
-      <parent link="${prefix}shooter_rightPanel_link" />
+      <parent link="${prefix}_shooter_rightPanel_link" />
       <child link="${prefix}_shooter_frontPanel_link" />
       <xacro:insert_block name="origin" />
     </joint>
+     <joint name="${prefix}_left_panel_joint" type="fixed">
+      <parent link="${prefix}_shooter_link" />
+      <child link="${prefix}_shooter_leftPanel_link" />
+      <xacro:insert_block name="origin" />
+    </joint>
+    <joint name="${prefix}_right_panel_joint" type="fixed">
+      <parent link="${prefix}_shooter_link" />
+      <child link="${prefix}_shooter_rightPanel_link" />
+      <xacro:insert_block name="origin" />
+    </joint>
+    <joint name="${prefix}_shooter_joint" type="fixed">
+     <parent link="${parent}"/>
+     <child link="${prefix}_shooter_link"/>
+     <xacro:insert_block name="origin"/>
+     </joint>
   </xacro:macro>
 </robot>

File: src/edna_description/urdf/robots/edna.urdf.xacro (robot description, xacro)
@@ -17,4 +17,5 @@
   <xacro:include filename="$(find edna_description)/urdf/parts/slider.xacro" />
   <xacro:include filename="$(find edna_description)/urdf/parts/intake.xacro" />
+  <xacro:include filename="$(find edna_description)/urdf/parts/shooter.xacro" />
   <xacro:include filename="$(find edna_description)/urdf/parts/versaroller.xacro" />
   <!-- Axle Position Variables -->
@@ -43,4 +44,7 @@
     <origin xyz="0 -0.46 0.09" rpy="0 0 0" />
   </xacro:intake>
+  <xacro:shooter parent="swerve_chassis_link" prefix="shooter">
+    <origin xyz="0 0 0" rpy="0 0 0" />
+  </xacro:shooter>
   <!-- Drive Train -->
   <xacro:swerve_axle prefix="front_left" parent="swerve_chassis_link">
