Commit message: Fixed shooter stl origin, moved collisions into one link in shooter xacro, general shooter changes

File: src/edna_description/urdf/parts/shooter.xacro (robot description, xacro)
@@ -1,6 +1,6 @@
-<?xml version="1.0" ?>
+<?xml version="1.0"?>
 <!--add 2 cylinders, with collisions wheel radius, and 4 revolute joints with panel-->
 <robot xmlns:xacro="http://www.ros.org/wiki/xacro">
-    <xacro:property name="panel_height" value="0.4266184" /> <!--also serves as back panel height-->
+    <!-- <xacro:property name="panel_height" value="0.4266184" /> also serves as back panel height
     <xacro:property name="panel_width" value="0.254" />
     <xacro:property name="panel_thick" value="0.00635" />
@@ -8,179 +8,121 @@
     <xacro:property name="back_panel_length" value="0.364" />
     <xacro:property name="back_panel_thick" value="0.021" />
-    <xacro:property name="back_panel_width" value="0.021" />
+    <xacro:property name="back_panel_width" value="0.021" /> -->
+    <!--<xacro:property name="wheel_length" value="0.025" /> --> <!--but really thickness-->
+    <!--<xacro:property name="back_panel_weight" value=""/>-->
+    <xacro:property name="mesh_x_offset" value="-0.03"/>
+    <xacro:property name="mesh_z_offset" value="0.053"/>
+    <xacro:property name="sidepanel_length" value="0.26" />
+    <xacro:property name="sidepanel_width" value="0.006" />
+    <xacro:property name="sidepanel_height" value="0.426" />
+    <xacro:property name="sidepanel_y_offset" value="0.186088" />
+    <xacro:property name="wheel_length" value="0.363538" />
     <xacro:property name="wheel_radius" value="0.0505" />
-    <!--<xacro:property name="wheel_length" value="0.025" /> --> <!--but really thickness-->
+    <xacro:property name="wheel_x_offset" value="0.08" /> <!-- This is a guess -->
+    <xacro:property name="wheel_z_offset" value="0.156" /> <!-- This is a guess -->
     <xacro:property name="wheel_mass" value="${0.11566605*4}" /> <!--not the most accurate, but issok-->
-    <xacro:property name="wheel_length" value="0.363538"/>
-    <!--<xacro:property name="back_panel_weight" value=""/>-->
-  <xacro:macro name="shooter" params="prefix parent *origin">
-    <link name="${prefix}_shooter_link">
-        <visual>
-            <origin xyz="0 0 0" rpy="${pi / 2} 0 0" />
-            <geometry>
-                <mesh filename="package://edna_description/meshes/RIFT_shooter.stl" scale="1 1 1" />
-            </geometry>
-            <material name="red" />
-        </visual>
-    </link>
-    <link name = "${prefix}_shooter_leftPanel_link">
-        <xacro:inertial_box mass = "${panel_weight}" x = "${panel_width}" y = "${panel_height}" z = "${panel_thick}">
-            <origin xyz = "0 0 0" rpy = "0 0 0"/>
-        </xacro:inertial_box>
-        <visual>
-            <origin xyz = "0 0 0" rpy = "0 0 0"/>
-            <geometry>
-                <box size="${panel_width} ${panel_height} ${panel_thick}"/>
-            </geometry>
-            <material name = "red"/>
-        </visual>
-        <collision>
-            <origin xyz = "0 0 0" rpy = "0 0 0"/>
-            <geometry>
-                <box size="${panel_width} ${panel_height} ${panel_thick}"/>
-            </geometry>
-        </collision>
-    </link>
-    <link name = "${prefix}_shooter_rightPanel_link">
-         <xacro:inertial_box mass = "${panel_weight}" x = "${panel_width}" y = "${panel_height}" z = "${panel_thick}">
-            <origin xyz = "0 0 0" rpy = "0 0 0"/>
-        </xacro:inertial_box>
-        <visual>
-            <origin xyz = "0 0 0" rpy = "0 0 0"/>
-            <geometry>
-                <box size="${panel_width} ${panel_height} ${panel_thick}"/>
-            </geometry>
-            <material name = "red"/>
-        </visual>
-        <collision>
-            <origin xyz = "0 0 0" rpy = "0 0 0"/>
-            <geometry>
-                <box size="${panel_width} ${panel_height} ${panel_thick}"/>
-            </geometry>
-        </collision>
-    </link>
-    <link name = "${prefix}_shooter_backPanel_link">
-        <xacro:inertial_box mass = "0.02" x = "${back_panel_length}" y = "${panel_height}" z = "${back_panel_thick}">
-            <origin xyz = "0 0 0" rpy = "0 0 0"/>
-        </xacro:inertial_box>
-        <visual>
-            <origin xyz = "0 0 0" rpy = "0 0 0"/>
-            <geometry>
-                <box size="${back_panel_width} ${panel_height} ${back_panel_thick}"/>
-            </geometry>
-            <material name = "red"/>
-        </visual>
-        <collision>
-            <origin xyz = "0 0 0" rpy = "0 0 0"/>
-            <geometry>
-                <box size="${back_panel_width} ${panel_height} ${back_panel_thick}"/>
-            </geometry>
-        </collision>
-    </link>
-    <link name = "${prefix}_shooter_frontPanel_link">
-        <xacro:inertial_box mass = "0.02" x = "${back_panel_length}" y = "${panel_height}" z = "${back_panel_thick}">
-            <origin xyz = "0 0 0" rpy = "0 0 0"/>
-        </xacro:inertial_box>
-        <visual>
-            <origin xyz = "0 0 0" rpy = "0 0 0"/>
-            <geometry>
-                <box size="${back_panel_width} ${panel_height} ${back_panel_thick}"/>
-            </geometry>
-            <material name = "red"/>
-        </visual>
-        <collision>
-            <origin xyz = "0 0 0" rpy = "0 0 0"/>
-            <geometry>
-                <box size="${back_panel_width} ${panel_height} ${back_panel_thick}"/>
-            </geometry>
-        </collision>
-    </link>
-    <link name="${prefix}_wheel_set1_link">
+    <xacro:macro name="shooter" params="prefix parent *origin">
+        <link name="${prefix}_link">
             <visual>
-                <origin xyz="0 0 0" rpy="${pi / 2} 0 0" />
+                <origin xyz="${mesh_x_offset} 0 ${mesh_z_offset}" rpy="0 ${pi/2} 0" />
                 <geometry>
-                    <mesh filename="" scale="0.001 0.001 0.001" />
+                    <mesh filename="package://edna_description/meshes/RiftShooter.stl" scale="1 1 1" />
                 </geometry>
                 <material name="red" />
             </visual>
             <collision>
-                <origin xyz="0 0 0" rpy="${pi / 2} 0 0"/>
+                <origin xyz="0 ${sidepanel_y_offset - sidepanel_width/2} 0" rpy="0 0 0" />
                 <geometry>
-                    <cylinder length="${wheel_length}" radius="${wheel_radius}"/>
-                    <!-- <mesh filename="package://edna_description/meshes/SwerveWheel.stl" scale="0.001 0.001 0.001" /> -->
+                    <box size="${sidepanel_length} ${sidepanel_width} ${sidepanel_height}" />
                 </geometry>
             </collision>
-            <xacro:inertial_cylinder mass="${wheel_mass}" radius="${wheel_radius}" length="${wheel_length}" >
+            <collision>
+                <origin xyz="0 ${-(sidepanel_y_offset - sidepanel_width/2)} 0" rpy="0 0 0" />
+                <geometry>
+                    <box size="${sidepanel_length} ${sidepanel_width} ${sidepanel_height}" />
+                </geometry>
+            </collision>
+        </link>
+        <link name="${prefix}_wheels_forward_link">
+            <collision>
+                <origin xyz="0 0 0" rpy="${pi / 2} 0 0" />
+                <geometry>
+                    <cylinder length="${wheel_length}" radius="${wheel_radius}" />
+                </geometry>
+            </collision>
+            <!-- Pretty sure something is wrong with this, but I don't know what... -->
+            <xacro:inertial_cylinder mass="${wheel_mass}" radius="${wheel_radius}" length="${wheel_length}">
                 <origin xyz="0 0 0" rpy="${pi / 2} 0 0" />
             </xacro:inertial_cylinder>
         </link>
-        <link name="${prefix}_wheel_set2_link">
-            <visual>
+        <link name="${prefix}_wheels_backward_link">
+            <collision>
                 <origin xyz="0 0 0" rpy="${pi / 2} 0 0" />
                 <geometry>
-                    <mesh filename="" scale="0.001 0.001 0.001" />
+                    <cylinder length="${wheel_length}" radius="${wheel_radius}" />
+                </geometry>
+            </collision>
+            <!-- Pretty sure something is wrong with this, but I don't know what... -->
+            <xacro:inertial_cylinder mass="${wheel_mass}" radius="${wheel_radius}" length="${wheel_length}">
+                <origin xyz="0 0 0" rpy="${pi / 2} 0 0" />
+            </xacro:inertial_cylinder>
+        </link>
+        <!-- <link name="${prefix}_backPanel_link">
+            <xacro:inertial_box mass="0.02" x="${back_panel_length}" y="${panel_height}"
+                z="${back_panel_thick}">
+                <origin xyz="0 0 0" rpy="0 0 0" />
+            </xacro:inertial_box>
+            <visual>
+                <origin xyz="0 0 0" rpy="0 0 0" />
+                <geometry>
+                    <box size="${back_panel_width} ${panel_height} ${back_panel_thick}" />
                 </geometry>
                 <material name="red" />
             </visual>
             <collision>
-                <origin xyz="0 0 0" rpy="${pi / 2} 0 0"/>
+                <origin xyz="0 0 0" rpy="0 0 0" />
                 <geometry>
-                    <cylinder length="${wheel_length}" radius="${wheel_radius}"/>
-                    <!-- <mesh filename="package://edna_description/meshes/SwerveWheel.stl" scale="0.001 0.001 0.001" /> -->
+                    <box size="${back_panel_width} ${panel_height} ${back_panel_thick}" />
                 </geometry>
             </collision>
-            <xacro:inertial_cylinder mass="${wheel_mass}" radius="${wheel_radius}" length="${wheel_length}" >
-                <origin xyz="0 0 0" rpy="${pi / 2} 0 0" />
-            </xacro:inertial_cylinder>
         </link>
-    <joint name="${prefix}_wheelset1_joint" type="revolute">
-      <origin xyz = "0 0 0" rpy = "0 0 0" />
-      <parent link="${prefix}_shooter_leftPanel_link"/>
-      <child link="${prefix}_wheel_set1_link"/>
-      <axis xyz = "0 1 0"/>
-      <limit effort="100" lower="-1" upper="1" velocity="2"/>
-    </joint>
-    <joint name="${prefix}_wheelset2_joint" type="revolute">
-      <origin xyz = "0 0 0" rpy = "0 0 0" />
-      <parent link="${prefix}_shooter_leftPanel_link"/>
-      <child link="${prefix}_wheel_set2_link"/>
-      <axis xyz = "0 1 0"/>
-      <limit effort="100" lower="-1" upper="1" velocity="2"/>
-    </joint>
-     <joint name="${prefix}_left_joint_back" type="fixed">
-      <parent link="${prefix}_shooter_leftPanel_link" />
-      <child link="${prefix}_shooter_backPanel_link" />
-      <xacro:insert_block name="origin" />
-    </joint>
-    <joint name="${prefix}_right_joint_back" type="fixed">
-      <parent link="${prefix}_shooter_rightPanel_link" />
-      <child link="${prefix}_shooter_backPanel_link" />
-      <xacro:insert_block name="origin" />
-    </joint>
-    <joint name="${prefix}_left_joint_front" type="fixed">
-      <parent link="${prefix}_shooter_leftPanel_link" />
-      <child link="${prefix}_shooter_frontPanel_link" />
-      <xacro:insert_block name="origin" />
-    </joint>
-    <joint name="${prefix}_right_joint_front" type="fixed">
-      <parent link="${prefix}_shooter_rightPanel_link" />
-      <child link="${prefix}_shooter_frontPanel_link" />
-      <xacro:insert_block name="origin" />
-    </joint>
-     <joint name="${prefix}_left_panel_joint" type="fixed">
-      <parent link="${prefix}_shooter_link" />
-      <child link="${prefix}_shooter_leftPanel_link" />
-      <xacro:insert_block name="origin" />
-    </joint>
-    <joint name="${prefix}_right_panel_joint" type="fixed">
-      <parent link="${prefix}_shooter_link" />
-      <child link="${prefix}_shooter_rightPanel_link" />
-      <xacro:insert_block name="origin" />
-    </joint>
-    <joint name="${prefix}_shooter_joint" type="fixed">
-     <parent link="${parent}"/>
-     <child link="${prefix}_shooter_link"/>
-     <xacro:insert_block name="origin"/>
-     </joint>
-  </xacro:macro>
+        <link name="${prefix}_frontPanel_link">
+            <xacro:inertial_box mass="0.02" x="${back_panel_length}" y="${panel_height}"
+                z="${back_panel_thick}">
+                <origin xyz="0 0 0" rpy="0 0 0" />
+            </xacro:inertial_box>
+            <visual>
+                <origin xyz="0 0 0" rpy="0 0 0" />
+                <geometry>
+                    <box size="${back_panel_width} ${panel_height} ${back_panel_thick}" />
+                </geometry>
+                <material name="red" />
+            </visual>
+            <collision>
+                <origin xyz="0 0 0" rpy="0 0 0" />
+                <geometry>
+                    <box size="${back_panel_width} ${panel_height} ${back_panel_thick}" />
+                </geometry>
+            </collision>
+        </link> -->
+        <joint name="${prefix}_joint" type="fixed">
+            <parent link="${parent}" />
+            <child link="${prefix}_link" />
+            <xacro:insert_block name="origin" />
+        </joint>
+        <joint name="${prefix}_wheels_forward_joint" type="fixed">
+            <origin xyz="${wheel_x_offset} 0 ${wheel_z_offset}" rpy="0 0 0" />
+            <parent link="${prefix}_link" />
+            <child link="${prefix}_wheels_forward_link" />
+            <axis xyz="0 1 0" />
+            <limit effort="100" lower="-1" upper="1" velocity="2" />
+        </joint>
+        <joint name="${prefix}_wheels_backward_joint" type="fixed">
+            <origin xyz="${-(wheel_x_offset - wheel_radius/2)} 0 ${wheel_z_offset}" rpy="0 0 0" />
+            <parent link="${prefix}_link" />
+            <child link="${prefix}_wheels_backward_link" />
+            <axis xyz="0 1 0" />
+            <limit effort="100" lower="-1" upper="1" velocity="2" />
+        </joint>
+    </xacro:macro>
 </robot>

File: src/edna_description/urdf/robots/edna.urdf.xacro (robot description, xacro)
@@ -45,6 +45,8 @@
     <origin xyz="0.46 0 0.09" rpy="0 0 ${pi/2}" />
   </xacro:intake>
-  <xacro:shooter parent="swerve_chassis_link" prefix="shooter">
-    <origin xyz="0 0 0" rpy="0 0 0" />
+  <!-- Shooter -->
+  <xacro:shooter prefix="shooter" parent="base_link">
+    <!-- <origin xyz="0 0 0" rpy="0 0 0" /> -->
+    <origin xyz="0.25 0 .33" rpy="0 ${-pi/6} 0" /> <!-- Made up values for shooter location & rotation. Change later. -->
   </xacro:shooter>
   <!-- Drive Train -->
