Commit message: switched out the mesh for regular box in arm.xacro

File: src/edna_description/urdf/parts/arm.xacro (robot description, xacro)
@@ -10,11 +10,13 @@
     <xacro:property name="arm_mount_height" value="0.0254" />
     <xacro:property name="arm_mount_weight" value="0.7589489" />
-    <xacro:macro name="armRift" params="parent *origin">
+    <xacro:macro name="arm" params="parent *origin">
         <!-- Left Bar Arm -->
         <link name="left_bar_link">
             <visual>
-                <origin xyz="0 0 0" rpy="0 0 0"/>
+                <origin xyz="${-arm_mount_width/2} 0 0" rpy="0 ${pi/2} ${pi/2}"/>
                 <geometry>
+                <!-- Mesh File doesnt work -->
                     <mesh filename="package://edna_description/meshes/ArmPart.stl" scale="1 1 1"/>
+                    <box size="${arm_bar_length} ${arm_bar_width} ${arm_bar_height}"/>
                 </geometry>
                 <material name="red"/>
@@ -26,7 +28,9 @@
         <link name="right_bar_link">
             <visual>
-                <origin xyz="${arm_mount_width} 0 0" rpy="0 0 0"/>
+            <origin xyz="${arm_mount_width/2} 0 0" rpy="0 ${pi/2} ${pi/2}"/>
                 <geometry>
+                <!-- Mesh File Does Not Work -->
                     <mesh filename="package://edna_description/meshes/ArmPart.stl" scale="1 1 1"/>
+                    <box size="${arm_bar_length} ${arm_bar_width} ${arm_bar_height}"/>
                 </geometry>
                 <material name="red"/>
@@ -38,7 +42,9 @@
         <link name="arm_mount_link">
             <visual>
-                <origin xyz="0 ${arm_bar_height} 0" rpy="0 0 0"/>
+                <origin xyz="0 ${arm_bar_height/2} 0" rpy="${pi/2} ${pi/2} 0"/>
                 <geometry>
+                <!-- Mesh File Does not Work -->
                     <mesh filename="package://edna_description/meshes/ShooterMount.stl" scale="1 1 1"/>
+                    <box size="${arm_mount_length} ${arm_mount_width} ${arm_mount_height}"/>
                 </geometry>
                 <material name="yellow"/>
@@ -48,5 +54,5 @@
         </link>
         <joint name="arm_mount_joint" type="fixed">
-            <origin xyz = "0 0 0" rpy = "0 0 0"/>
+            <origin xyz = "0 0 .2" rpy = "0 0 0"/>
             <parent link="${parent}"/>
             <child link="arm_mount_link"/>

File: src/edna_description/urdf/parts/intake.xacro (robot description, xacro)
@@ -4,5 +4,5 @@
     <link name="intake_link">
         <visual>
-            <origin xyz="0 0 0" rpy="0 0 0" />
+            <origin xyz="0 0 0" rpy="0 {pi}/2 0" />
             <geometry>
                 <mesh filename="package://edna_description/meshes/RiftIntake.stl" scale="1 1 1" />

File: src/edna_description/urdf/robots/edna.urdf.xacro (robot description, xacro)
@@ -19,4 +19,5 @@
   <xacro:include filename="$(find edna_description)/urdf/parts/shooter.xacro" />
   <xacro:include filename="$(find edna_description)/urdf/parts/versaroller.xacro" />
+  <xacro:include filename="$(find edna_description)/urdf/parts/arm.xacro" />
   <!-- Axle Position Variables -->
   <xacro:property name="axle_pos" value="0.261523" />
@@ -41,4 +42,8 @@
     <origin xyz="0 0 0" rpy="0 0 0" />
   </xacro:square_chassis>
+  <!-- Arm -->
+  <xacro:arm parent="base_link">
+    <origin xyz="0 0 0" rpy="0 0 0" />
+  </xacro:arm>
   <!-- Intake -->
   <xacro:intake parent="swerve_chassis_link">
